File: IC-SDC-Hub V2.3/IC-SDC-Hub V2.3.kicad_pcb (KiCad board)
At the start: 2 copper layers, 58 x 78 mm, 33 parts, among them J1 JST-XA, J10 JST-XA, J11 JST-XA, J2 JST-XA, J3 JST-XA, J4 JST-XA, J5 JST-XA, J6 JST-XA, J7 Conn_01x03, J8 Conn_01x03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

Commit message: final pcb I think
Parts:
- renumbered BSPD to D1, COCK to D2, LEFT to D3, RIGHT to D4, BOTS to D5, IS to D6
Connections:
- U1 pad 11: unconnected-(U1-Pad11) -> GND
Routing:
- net BSPD_S: track 27.5 -> 29.8 mm
- net BOTS_S: track 48.7 -> 51.0 mm
- net IS_S: track 52.3 -> 54.5 mm
- net CK_S: track 31.1 -> 33.3 mm
- net L_S: track 34.6 -> 36.9 mm
- net R_S: track 40.1 -> 42.3 mm

Commit message: Ready to order
Parts:
- added REF**: jamesp-F.Cu, CustomFootprints:jamesp-F.Cu, F.Cu at (226.0, 130.0)
- renumbered D5 to BOTS, D1 to BSPD, D2 to CKPT, D6 to IS, D3 to LEFT, D4 to RIGHT
Other:
- board text added: "(sense)"
